File: hardware/backplane/power.kicad_sch (KiCad schematic)
At the start: 11 parts, among them U4 SC189BULTRT, U5 TPS62132

Commit message: feat: Assign footprints, add testpoints
 * Verify all footprints are assigned.
 * Create testpoints for key signals.
 * Reorganize component libraries.
Parts:
- added TP1: +1V1, TestPoint:TestPoint_Keystone_5000-5004_Miniature, symbol Connector:TestPoint
- added TP14, TP15, TP16, TP17: GND, TestPoint:TestPoint_Keystone_5000-5004_Miniature, symbol Connector:TestPoint
- added TP2: +3V3, TestPoint:TestPoint_Keystone_5000-5004_Miniature, symbol Connector:TestPoint
- added TP3: PG, TestPoint:TestPoint_Pad_D1.0mm, symbol Connector:TestPoint
- C4, C7: footprint (none) -> Capacitor_SMD:C_0805_2012Metric; Part Number (none) -> GRM21BR71A106KA73L
- C5, C9: footprint (none) -> Capacitor_SMD:C_0805_2012Metric; Part Number (none) -> GRM21BR60J226ME39K
- C6: value 3 nF -> 3.3 nF; footprint (none) -> Capacitor_SMD:C_0402_1005Metric; Part Number (none) -> GRM155R71C104KA88J
- C8: footprint (none) -> Capacitor_SMD:C_0402_1005Metric; Part Number (none) -> GRM155R71C104KA88J
- L1: value 1 µH -> 2.2 µH; footprint (none) -> Inductor_SMD:L_Bourns_SRN6045TA; Part Number (none) -> HPC 6045NC-2R2M
- L2: footprint (none) -> Inductor_SMD:L_Bourns_SRN6045TA; Part Number (none) -> HPC 6045NC-2R2M
- R15: footprint (none) -> Resistor_SMD:R_0402_1005Metric; Part Number (none) -> RC0402FR-07100KL
- U4: footprint (none) -> SC189x:MLPD-UT6; Part Number (none) -> SC189BULTRT
- U5: Part Number (none) -> TPS62132RGTR
Connections:
- net +1V1: now also TP1.1
- net +3V3: now also TP2.1
- net GND: now also TP14.1, TP15.1, TP16.1, TP17.1
- net PG: now also TP3.1
Other:
- moved on the sheet: C4, C5, C6, C7, C8, C9, L1, L2, R15, U4, U5
