File: hardware/backplane/rclk_fanout.kicad_sch (KiCad schematic)
At the start: 8 parts, among them U11 PL133-97QC-R, U12 PL133-97QC-R

Commit message: feat: Assign footprints, add testpoints
 * Verify all footprints are assigned.
 * Create testpoints for key signals.
 * Reorganize component libraries.
Parts:
- removed RN4, RN5: 33 Ω, symbol Device:R_Pack05
- added RN4, RN5: 33 Ω, YC248-JR-0733RL:RES_YC248_4X1P6_YAG, symbol Device:R_Pack08
- added TP22: RCLK, TestPoint:TestPoint_Pad_D1.0mm, symbol Connector:TestPoint
- C21, C22, C23, C24: footprint (none) -> Capacitor_SMD:C_0402_1005Metric; Part Number (none) -> GRM155R71C104KA88J
- U11, U12: footprint QFN-16_MCL -> Package_DFN_QFN:QFN-16-1EP_3x3mm_P0.5mm_EP1.7x1.7mm; Part Number (none) -> PL133-97QC
Connections:
- net RCLK: now also TP22.1
- net RCLK0: now also RN4.5 (R5.1)
- net RCLK1: now also RN4.4 (R4.1)
- net RCLK2: now also RN4.3 (R3.1)
- net RCLK3: now also RN4.2 (R2.1)
- net RCLK4: now also RN4.1 (R1.1)
- net RCLK5: now also RN5.5 (R5.1)
- net RCLK6: now also RN5.4 (R4.1)
- net RCLK7: now also RN5.3 (R3.1)
- net RCLK8: now also RN5.2 (R2.1)
- net RCLK9: now also RN5.1 (R1.1)
- net at U12.9 (CLK5): now also RN5.12 (R5.2)
- net at U12.8 (CLK4): now also RN5.13 (R4.2)
- net at U12.5 (CLK3): now also RN5.14 (R3.2)
- net at U12.4 (CLK2): now also RN5.15 (R2.2)
- net at U12.1 (CLK1): now also RN5.16 (R1.2)
- net at U11.1 (CLK1): now also RN4.16 (R1.2)
- net at U11.12 (CLK6): now also RN4.11 (R6.2)
- net at U11.13 (CLK7): now also RN4.10 (R7.2)
- net at U11.14 (CLK8): now also RN4.9 (R8.2)
- net at U11.4 (CLK2): now also RN4.15 (R2.2)
- net at U11.5 (CLK3): now also RN4.14 (R3.2)
- net at U11.8 (CLK4): now also RN4.13 (R4.2)
- net at U11.9 (CLK5): now also RN4.12 (R5.2)
- net at U12.12 (CLK6): now also RN5.11 (R6.2)
- net at U12.13 (CLK7): now also RN5.10 (R7.2)
- net at U12.14 (CLK8): now also RN5.9 (R8.2)
