File: hardware/backplane/usb.kicad_sch (KiCad schematic)
At the start: 22 parts, among them J1 USB_C_Receptacle_USB2.0_16P, U1 USBLC6-2SC6, U2 UTC2000/MG, U3 NCP360SN

Commit message: feat: Assign footprints, add testpoints
 * Verify all footprints are assigned.
 * Create testpoints for key signals.
 * Reorganize component libraries.
Parts:
- removed J1: USB_C_Receptacle_USB2.0_16P, symbol Connector:USB_C_Receptacle_USB2.0_16P
- added J1: USB-C, USB4215-03-A:GCT_USB4215-03-A_REVA, symbol USB4215-03-A_REVA:USB4215-03-A_REVA
- added TP10: ~{0.5A}, TestPoint:TestPoint_Pad_D1.0mm, symbol Connector:TestPoint
- added TP11: FAULT, TestPoint:TestPoint_Pad_1.0x1.0mm, symbol Connector:TestPoint
- added TP12: ~{CONN}, TestPoint:TestPoint_Pad_1.0x1.0mm, symbol Connector:TestPoint
- added TP13: VSUP, TestPoint:TestPoint_Keystone_5000-5004_Miniature, symbol Connector:TestPoint
- added TP4: VBUS, TestPoint:TestPoint_Keystone_5000-5004_Miniature, symbol Connector:TestPoint
- added TP5: ~{OCS}, TestPoint:TestPoint_Pad_1.0x1.0mm, symbol Connector:TestPoint
- added TP6: VMON, TestPoint:TestPoint_Pad_1.0x1.0mm, symbol Connector:TestPoint
- added TP8: ~{3.0A}, TestPoint:TestPoint_Pad_D1.0mm, symbol Connector:TestPoint
- added TP9: ~{1.5A}, TestPoint:TestPoint_Pad_D1.0mm, symbol Connector:TestPoint
- C1: footprint (none) -> Capacitor_SMD:C_0402_1005Metric; Part Number (none) -> GRM155R71C104KA88J
- C2, C3: footprint (none) -> Capacitor_SMD:C_0603_1608Metric; Part Number (none) -> CC0603KRX7R7BB105
- D1: value USB Fault -> Red; footprint (none) -> LED_SMD:LED_0603_1608Metric; Indicates (none) -> USB Fault; Part Number (none) -> 150060RS55040
- R1, R2, R5: footprint (none) -> Resistor_SMD:R_0402_1005Metric; Part Number (none) -> CR0402-FX-5101GLF
- R10, R12, R13, R14, R3, R4, R7, R8, R9: footprint (none) -> Resistor_SMD:R_0402_1005Metric; Part Number (none) -> CR0402-JW-103GLF
- R11: footprint (none) -> Resistor_SMD:R_0402_1005Metric; Part Number (none) -> RMCF0402FT510R
- R6: footprint (none) -> Resistor_SMD:R_0402_1005Metric; Part Number (none) -> RMCF0402FT35K7
- U1: Part Number (none) -> USBLC6-2SC6
- U2: footprint QFN16_3X3X0.9_MCH -> Package_DFN_QFN:VQFN-16-1EP_3x3mm_P0.5mm_EP1.1x1.1mm; Part Number (none) -> UTC2000/MG
- U3: Part Number (none) -> NCP360SNT1G
Connections:
- net GND: now also J1.A1_B12 (GND_A), J1.B1_A12 (GND_B), J1.SH1 (SHIELD), J1.SH2 (SHIELD), J1.SH3 (SHIELD), J1.SH4 (SHIELD)
- net VBUS: now also J1.A4_B9 (VBUS_A), J1.B4_A9 (VBUS_B), TP4.1
- net VSUP: now also TP13.1
- net ~{0.5A}: now also TP10.1
- net ~{1.5A}: now also TP9.1
- net ~{3.0A}: now also TP8.1
- net at R2.1, R3.1: now also J1.A5 (CC1)
- net at U1.3 (I/O2): now also J1.A6 (DP1), J1.B6 (DP2)
- net at U1.1 (I/O1): now also J1.A7 (DN1), J1.B7 (DN2)
- net at R1.1, R4.1: now also J1.B5 (CC2)
- net at R5.2, R6.1, U2.12 (VMON): now also TP6.1
- net at R11.1, U2.4 (FAULT_IND): now also TP11.1
- net at R10.2, U2.5 (AUDIO_ADAPTER/CONNECTED#), U3.3 (~{EN}): now also TP12.1
- net at R9.2, U2.1 (OCS#), U3.4 (~{FLAG}): now also TP5.1
Other:
- moved on the sheet: R1, R2, R3, R4, U1
