File: hardware/backplane/control_port.kicad_sch (KiCad schematic)
At the start: 1 part, among them J20 SFH11-PBPC-D13-RA-BK

Commit message: feat: Assign footprints, add testpoints
 * Verify all footprints are assigned.
 * Create testpoints for key signals.
 * Reorganize component libraries.
Parts:
- J20: value SFH11-PBPC-D13-RA-BK -> Control; Part Number (none) -> SFH11-PBPC-D13-RA-BK
Changed lines of the file:
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@@
 			)
 		)
-		(property "Value" "SFH11-PBPC-D13-RA-BK"
+		(property "Value" "Control"
 			(at 135.89 120.65 0)
 			(effects
@@
 			)
 		)
-		(property "Datasheet" "~"
+		(property "Datasheet" "https://s3.amazonaws.com/catalogspreads-pdf/PAGE123%20.100%20SFH11%20SERIES%20FEMALE%20HDR%20ST%20RA.pdf"
 			(at 134.62 101.6 0)
 			(effects
@@
 			(at 134.62 101.6 0)
 			(effects
+				(font
+					(size 1.27 1.27)
+				)
+				(hide yes)
+			)
+		)
+		(property "Indicates" ""
+			(at 134.62 101.6 0)
+			(effects
+				(font
+					(size 1.27 1.27)
+				)
+				(hide yes)
+			)
+		)
+		(property "Part Number" "SFH11-PBPC-D13-RA-BK"
+			(at 134.62 101.6 0)
+			(effects

Commit message: feat: Apply bus arch changes to backplane schematic
Connections:
- net ~{CPURST} renamed ~{CRST}
Changed lines of the file:
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@@
 		)
 	)
-	(hierarchical_label "~{CPURST}"
+	(hierarchical_label "~{CRST}"
 		(shape bidirectional)
 		(at 157.48 109.22 0)
