File: hardware/backplane/mclk_fanout.kicad_sch (KiCad schematic)
At the start: 12 parts, among them U10 PL133-97QC-R, U8 PL133-97QC-R, U9 PL133-97QC-R

Commit message: feat: Re-add peripheral MCLK, add to memory lines (#3)
Need MCLK to maintain peripheral synchronization.  Add missing memory
access size and latch lines.
Connections:
- net MCLK10: now also RN3.6 (R6.1); no longer RN3.12 (R1.2)
- net MCLK11: now also RN3.5 (R5.1); no longer RN3.11 (R2.2)
- net MCLK12: now also RN3.4 (R4.1); no longer RN3.10 (R3.2)
- net MCLK13: now also RN3.3 (R3.1); no longer RN3.9 (R4.2)
- net MCLK14: now also RN3.2 (R2.1); no longer RN3.8 (R5.2)
- net MCLK15: now also RN3.1 (R1.1); no longer RN3.7 (R6.2)
- net at U10.12 (CLK6): now also RN3.7 (R6.2); no longer RN3.1 (R1.1)
- net at U10.9 (CLK5): now also RN3.8 (R5.2); no longer RN3.2 (R2.1)
- net at U10.8 (CLK4): now also RN3.9 (R4.2); no longer RN3.3 (R3.1)
- net at U10.5 (CLK3): now also RN3.10 (R3.2); no longer RN3.4 (R4.1)
- net at U10.4 (CLK2): now also RN3.11 (R2.2); no longer RN3.5 (R5.1)
- net at U10.1 (CLK1): now also RN3.12 (R1.2); no longer RN3.6 (R6.1)
Other:
- moved on the sheet: C15, C16, C18, C19, RN1, RN2, U8, U9

Commit message: feat: Assign footprints, add testpoints
 * Verify all footprints are assigned.
 * Create testpoints for key signals.
 * Reorganize component libraries.
Parts:
- removed RN1, RN2: 33 Ω, symbol Device:R_Pack05
- removed RN3: 33 Ω, symbol Device:R_Pack06
- added RN1, RN2, RN3: 33 Ω, YC248-JR-0733RL:RES_YC248_4X1P6_YAG, symbol Device:R_Pack08
- added TP21: MCLK, TestPoint:TestPoint_Pad_D1.0mm, symbol Connector:TestPoint
- C15, C16, C17, C18, C19, C20: footprint (none) -> Capacitor_SMD:C_0402_1005Metric; Part Number (none) -> GRM155R71C104KA88J
- U10, U8, U9: footprint QFN-16_MCL -> Package_DFN_QFN:QFN-16-1EP_3x3mm_P0.5mm_EP1.7x1.7mm; Part Number (none) -> PL133-97QC
Connections:
- net MCLK: now also TP21.1
- net MCLK0: now also RN1.5 (R5.1)
- net MCLK1: now also RN1.4 (R4.1)
- net MCLK10: now also RN3.6 (R6.1)
- net MCLK11: now also RN3.5 (R5.1)
- net MCLK12: now also RN3.4 (R4.1)
- net MCLK13: now also RN3.3 (R3.1)
- net MCLK14: now also RN3.2 (R2.1)
- net MCLK15: now also RN3.1 (R1.1)
- net MCLK2: now also RN1.3 (R3.1)
- net MCLK3: now also RN1.2 (R2.1)
- net MCLK4: now also RN1.1 (R1.1)
- net MCLK5: now also RN2.5 (R5.1)
- net MCLK6: now also RN2.4 (R4.1)
- net MCLK7: now also RN2.3 (R3.1)
- net MCLK8: now also RN2.2 (R2.1)
- net MCLK9: now also RN2.1 (R1.1)
- net at U9.9 (CLK5): now also RN2.12 (R5.2)
- net at U9.8 (CLK4): now also RN2.13 (R4.2)
- net at U9.5 (CLK3): now also RN2.14 (R3.2)
- net at U9.4 (CLK2): now also RN2.15 (R2.2)
- net at U9.1 (CLK1): now also RN2.16 (R1.2)
- net at U8.9 (CLK5): now also RN1.12 (R5.2)
- net at U8.8 (CLK4): now also RN1.13 (R4.2)
- net at U8.5 (CLK3): now also RN1.14 (R3.2)
- net at U8.4 (CLK2): now also RN1.15 (R2.2)
- net at U8.1 (CLK1): now also RN1.16 (R1.2)
- net at U9.12 (CLK6): now also RN2.11 (R6.2)
- net at U9.13 (CLK7): now also RN2.10 (R7.2)
- net at U9.14 (CLK8): now also RN2.9 (R8.2)
- net at U10.5 (CLK3): now also RN3.14 (R3.2)
- net at U10.4 (CLK2): now also RN3.15 (R2.2)
- net at U10.1 (CLK1): now also RN3.16 (R1.2)
- net at U10.12 (CLK6): now also RN3.11 (R6.2)
- net at U10.9 (CLK5): now also RN3.12 (R5.2)
- net at U10.8 (CLK4): now also RN3.13 (R4.2)
- net at U10.13 (CLK7): now also RN3.10 (R7.2)
- net at U10.14 (CLK8): now also RN3.9 (R8.2)
- net at U8.12 (CLK6): now also RN1.11 (R6.2)
- net at U8.13 (CLK7): now also RN1.10 (R7.2)
- net at U8.14 (CLK8): now also RN1.9 (R8.2)

Commit message: feat: Apply bus arch changes to backplane schematic
Connections:
- net ~{CPURST} renamed ~{CRST}
Changed lines of the file:
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@@
 		)
 	)
-	(hierarchical_label "~{CPURST}"
+	(hierarchical_label "~{CRST}"
 		(shape input)
 		(at 26.67 44.45 180)
